File: pcb/rev.A/mist1010.kicad_pcb (KiCad board)
At the start: 2 copper layers, 100 x 100 mm, 206 parts, among them J1 Conn_02x05_Odd_Even, J10 TE 041021-4, J11 Conn_01x03, J12 Conn_01x04, J13 Conn_02x05_Odd_Even, J14 Conn_02x05_Odd_Even, J15 Conn_01x04, J16 MEM2055-00-190-01-A, J17 Conn_01x04, J2 USB_B_Micro, J3 Conn_02x05_Odd_Even, J4 PJ-320D, J5 USB_A, J6 USB_A, J7 USB_A, J8 USB_A, J9 DB15_Female_HighDensity_Mount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, Q1 IRLML6402, Q2 IRLML6402, Q3 BC817, Q4 BC817, SW1 Jumper / Pin header 1x2 Pitch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, SW2 SW_DIP_x02, SW3 SW_Push, SW4 SW_Push, SW5 SW_Push, U1 MT48LC16M16A2, U10 LD1117AS25TR, U2 AT91SAM7S256-AU, U3 EP3C25E144, U4 MAX3421E, U5 FE2.1-LQFP48, U6 ATtiny45-20PU, U7 DS1307Z+, U8 LM3940IS-3.3, U9 LD1117AS12TR, X1 27 MHz, X2 12 MHz, Y1 18.432 MHz, Y2 32768 Hz

Commit message: update pcb rev.A
Parts:
- D1: value LED_RED -> LED_Red
- D2: value LED_YELLOW -> LED_Yellow
- D3: value LED_GREEN -> LED_Green
- J16: moved to F.Cu
- J4: value PJ-320D -> PJ-320
- moved J1 10.5 mm to (172.9, 114.7), turned to 180 degrees
- moved J13 10.5 mm to (107.4, 71.5), turned to 0 degrees
- moved J14 10.5 mm to (179.9, 122.8), turned to 0 degrees
- moved J3 10.5 mm to (179.9, 104.5), turned to 0 degrees
- moved J11 5.12 mm to (120.4, 60.8), turned to 0 degrees
- moved R69 4.16 mm to (184.9, 127.4)
- moved R70 4.16 mm to (184.9, 131.6)
- moved R71 4.16 mm to (177.4, 127.4)
- moved R72 4.16 mm to (177.4, 131.6)
- moved D1 2.00 mm to (128.3, 142.5)
- moved D2 2.00 mm to (115.0, 142.5)
- moved D3 2.00 mm to (101.8, 142.5)
- moved R45 2.00 mm to (129.5, 139.8)
- moved R46 2.00 mm to (116.3, 139.8)
- moved R47 2.00 mm to (103.1, 139.8)
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Connections:
- J11 pad 1: /TAPE_OUT -> GND
- J11 pad 3: GND -> /TAPE_OUT
Routing:
- net GND: track 483.1 -> 526.4 mm, vias 374 -> 384
- net /SS1: track 49.5 -> 33.3 mm
- net /SD_DAT2: track 32.1 -> 16.9 mm
- net /MOSI: track 111.0 -> 95.9 mm, vias 8 -> 7
- net /~JOY1_DOWN: track 39.1 -> 52.6 mm
- net /SD_CD: track 50.2 -> 37.5 mm, vias 3 -> 2
- net /~JOY0_UP: track 9.01 -> 21.7 mm, vias 0 -> 2
- net /SD_DAT1: track 25.2 -> 14.7 mm, vias 2 -> 1
- net /~JOY0_LEFT: track 13.7 -> 22.7 mm
- net /FPGA_TDI: track 35.8 -> 26.9 mm, vias 3 -> 2
- net /MISO: track 109.7 -> 101.4 mm, vias 5 -> 4
- net /~JOY0_DOWN: track 10.3 -> 18.1 mm, vias 1 -> 0
- net +3V3: track 722.5 -> 729.9 mm, vias 47 -> 44
- net /ARM_TMS: track 58.2 -> 51.1 mm, vias 2 -> 1
- net Net-(J1-Pad7): track 26.4 -> 19.4 mm, vias 2 -> 0
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
Commit message: update pcb rev.A
Parts:
- added C75: 10u, Capacitor_SMD:C_0805_2012Metric_Pad1.18x1.45mm_HandSolder, B.Cu at (123.6, 66.0)
- added C76: 10u, Capacitor_SMD:C_0805_2012Metric_Pad1.18x1.45mm_HandSolder, B.Cu at (123.7, 80.2)
- added C77: 100n, Capacitor_SMD:C_0603_1608Metric_Pad1.08x0.95mm_HandSolder, B.Cu at (131.4, 64.3)
- added C78: 100n, Capacitor_SMD:C_0603_1608Metric_Pad1.08x0.95mm_HandSolder, B.Cu at (137.4, 74.8)
- added C79: 100n, Capacitor_SMD:C_0603_1608Metric_Pad1.08x0.95mm_HandSolder, B.Cu at (134.4, 69.4)
- added C80: 220u, Capacitor_Tantalum_SMD:CP_EIA-7343-31_Kemet-D, B.Cu at (131.3, 73.0)
- added C81: 10p, Capacitor_SMD:C_0603_1608Metric_Pad1.08x0.95mm_HandSolder, B.Cu at (114.8, 69.8)
- added L4: 1u, Inductor_SMD:L_0805_2012Metric_Pad1.15x1.40mm_HandSolder, B.Cu at (134.7, 79.3)
- added R101: 75, Resistor_SMD:R_0603_1608Metric_Pad0.98x0.95mm_HandSolder, B.Cu at (132.9, 64.3)
- added R102: 75, Resistor_SMD:R_0603_1608Metric_Pad0.98x0.95mm_HandSolder, B.Cu at (138.9, 74.8)
- added R103: 75, Resistor_SMD:R_0603_1608Metric_Pad0.98x0.95mm_HandSolder, B.Cu at (135.9, 69.4)
- added R76: 1k, Resistor_SMD:R_0603_1608Metric_Pad0.98x0.95mm_HandSolder, B.Cu at (143.9, 64.3)
- added R77: 1.1k, Resistor_SMD:R_0603_1608Metric_Pad0.98x0.95mm_HandSolder, B.Cu at (142.4, 64.3)
- added R78: 1.1k, Resistor_SMD:R_0603_1608Metric_Pad0.98x0.95mm_HandSolder, B.Cu at (140.7, 64.3)
- added R79: 2.2k, Resistor_SMD:R_0603_1608Metric_Pad0.98x0.95mm_HandSolder, B.Cu at (139.2, 64.3)
- added R80: 4.3k, Resistor_SMD:R_0603_1608Metric_Pad0.98x0.95mm_HandSolder, B.Cu at (137.7, 64.3)
- added R81: 9.1k, Resistor_SMD:R_0603_1608Metric_Pad0.98x0.95mm_HandSolder, B.Cu at (136.2, 64.3)
- added R82: 18k, Resistor_SMD:R_0603_1608Metric_Pad0.98x0.95mm_HandSolder, B.Cu at (134.7, 64.3)
- added R83: 1k, Resistor_SMD:R_0603_1608Metric_Pad0.98x0.95mm_HandSolder, B.Cu at (149.7, 74.8)
- added R84: 1.1k, Resistor_SMD:R_0603_1608Metric_Pad0.98x0.95mm_HandSolder, B.Cu at (148.2, 74.8)
- added R85: 1.1k, Resistor_SMD:R_0603_1608Metric_Pad0.98x0.95mm_HandSolder, B.Cu at (146.7, 74.8)
- added R86: 2.2k, Resistor_SMD:R_0603_1608Metric_Pad0.98x0.95mm_HandSolder, B.Cu at (145.2, 74.8)
- added R87: 4.3k, Resistor_SMD:R_0603_1608Metric_Pad0.98x0.95mm_HandSolder, B.Cu at (143.7, 74.8)
- added R88: 9.1k, Resistor_SMD:R_0603_1608Metric_Pad0.98x0.95mm_HandSolder, B.Cu at (142.2, 74.8)
- added R89: 75, Resistor_SMD:R_0603_1608Metric_Pad0.98x0.95mm_HandSolder, B.Cu at (127.2, 64.3)
- added R90: 18k, Resistor_SMD:R_0603_1608Metric_Pad0.98x0.95mm_HandSolder, B.Cu at (140.7, 74.8)
- added R91: 1k, Resistor_SMD:R_0603_1608Metric_Pad0.98x0.95mm_HandSolder, B.Cu at (146.9, 69.4)
- added R92: 1.1k, Resistor_SMD:R_0603_1608Metric_Pad0.98x0.95mm_HandSolder, B.Cu at (145.4, 69.4)
- added R93: 1.1k, Resistor_SMD:R_0603_1608Metric_Pad0.98x0.95mm_HandSolder, B.Cu at (143.7, 69.4)
- added R94: 2.2k, Resistor_SMD:R_0603_1608Metric_Pad0.98x0.95mm_HandSolder, B.Cu at (142.2, 69.4)
- added R95: 4.3k, Resistor_SMD:R_0603_1608Metric_Pad0.98x0.95mm_HandSolder, B.Cu at (140.7, 69.4)
- added R96: 9.1k, Resistor_SMD:R_0603_1608Metric_Pad0.98x0.95mm_HandSolder, B.Cu at (139.2, 69.4)
- added R97: 18k, Resistor_SMD:R_0603_1608Metric_Pad0.98x0.95mm_HandSolder, B.Cu at (137.7, 69.4)
- added R98: 4.7M, Resistor_SMD:R_0603_1608Metric_Pad0.98x0.95mm_HandSolder, B.Cu at (116.3, 69.8)
- added U11: AD724, Package_SO:SOIC-16W_7.5x10.3mm_P1.27mm, B.Cu at (123.3, 73.3)
- added Y3: 4.433619 MHz, Crystal:Crystal_SMD_5032-2Pin_5.0x3.2mm, B.Cu at (115.6, 74.6)
Connections:
- J4 pad S: unconnected-(J4-PadS) -> (no net)
Routing:
- net Net-(C75-Pad2): track 0.00 -> 32.8 mm
- net Net-(C78-Pad1): track 0.00 -> 14.4 mm
- net /AUDIO_L: track 54.2 -> 67.4 mm
- net Net-(C77-Pad2): track 0.00 -> 12.5 mm
- net Net-(C79-Pad2): track 0.00 -> 12.5 mm
- net Net-(C78-Pad2): track 0.00 -> 12.3 mm
- net +5V: track 195.0 -> 207.2 mm, vias 10 -> 11
- net /AUDIO_R: track 39.7 -> 51.8 mm
- net Net-(R14-Pad2): track 33.7 -> 45.7 mm
- net Net-(C81-Pad1): track 0.00 -> 11.2 mm
- net Net-(C77-Pad1): track 0.00 -> 11.1 mm, vias 0 -> 2
- net /VGA_HS: track 45.0 -> 55.0 mm, vias 2 -> 3
- net Net-(C79-Pad1): track 0.00 -> 9.15 mm
- net GND: track 526.4 -> 534.3 mm, vias 384 -> 381
- net Net-(C80-Pad2): track 0.00 -> 7.01 mm
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
Commit message: update pcb rev.A
Parts:
- C75, C76, C77, C78, C79, C80, C81, L4, R101, R102, R103, R98, U11: moved to F.Cu
- R15, R16, R17, R18, R19, R20, R21, R22, R23, R25, R26, R28, R31, R32, R33, R34, R35, R37, R39, R40, R41, R42, R43: moved to B.Cu
- Y3: footprint Crystal:Crystal_SMD_5032-2Pin_5.0x3.2mm -> Crystal:Crystal_SMD_HC49-SD; moved to F.Cu
- moved C81 37.7 mm to (152.2, 64.7), turned to -90 degrees
- moved R98 36.9 mm to (152.2, 61.4)
- moved Y3 31.4 mm to (144.4, 62.4), turned to 180 degrees
- moved C75 28.1 mm to (151.4, 69.8), turned to 90 degrees
- moved U11 21.1 mm to (144.2, 70.6), turned to 0 degrees
- moved C76 19.0 mm to (142.4, 77.1), turned to 0 degrees
- moved L4 11.7 mm to (146.2, 77.1)
- moved C80 9.62 mm to (134.9, 64.1)
- moved R89 9.08 mm to (134.9, 59.6), turned to 0 degrees
- moved R82 8.40 mm to (126.5, 62.5)
- moved R103 7.70 mm to (134.9, 77.0), turned to 180 degrees
- moved R97 7.52 mm to (130.2, 68.3), turned to -90 degrees
- moved R90 7.52 mm to (133.2, 73.8)
- moved R101 6.97 mm to (134.9, 71.0), turned to 180 degrees
- moved R21 6.95 mm to (128.0, 62.5)
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Connections:
- net Net-(C75-Pad2) renamed +5V_PAL
- J4 pad S: (no net) -> /Composite
- R89 pad 1: (no net) -> /Composite
Routing:
- net Net-(C77-Pad2): track 12.5 -> 33.5 mm, vias 0 -> 1
- net Net-(C79-Pad2): track 12.5 -> 33.0 mm, vias 0 -> 1
- net /G: track 26.3 -> 41.5 mm
- net Net-(C78-Pad2): track 12.3 -> 25.0 mm, vias 0 -> 1
- net Net-(C80-Pad1): track 6.21 -> 18.5 mm, vias 0 -> 2
- net /R: track 16.0 -> 26.8 mm
- net Net-(C78-Pad1): track 14.4 -> 4.27 mm
- net /Composite: track 0.00 -> 9.23 mm
- net +5V: track 207.2 -> 198.9 mm, vias 11 -> 10
- net /VGA_R0: track 44.4 -> 52.7 mm, vias 2 -> 1
- net /B: track 25.4 -> 33.3 mm
- net +5V_PAL: track 32.8 -> 25.5 mm
- net /VGA_B0: track 35.2 -> 41.2 mm, vias 2 -> 1
- net Net-(C81-Pad1): track 11.2 -> 17.2 mm
- net Net-(C80-Pad2): track 7.01 -> 1.76 mm, vias 0 -> 1
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Other:
- board text added: "PAL"
- board text added: "VGA"
