File: pcb/rev.A/mist1010.kicad_pcb (KiCad board)
At the start: 2 copper layers, 100 x 100 mm, 242 parts, among them J1 Conn_02x05_Odd_Even, J10 TE 041021-4, J11 Conn_01x03, J12 Conn_01x04, J13 Conn_02x05_Odd_Even, J14 Conn_02x05_Odd_Even, J15 Conn_01x04, J16 MEM2055-00-190-01-A, J17 Conn_01x04, J2 USB_B_Micro, J3 Conn_02x05_Odd_Even, J4 PJ-320, J5 USB_A, J6 USB_A, J7 USB_A, J8 USB_A, J9 DB15_Female_HighDensity_Mount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, Q1 IRLML6402, Q2 IRLML6402, Q3 BC817, Q4 BC817, SW1 Jumper / Pin header 1x2 Pitch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, SW2 SW_DIP_x02, SW3 SW_Push, SW4 SW_Push, SW5 SW_Push, U1 MT48LC16M16A2, U10 LD1117AS25TR, U11 AD724, U2 AT91SAM7S256-AU, U3 EP3C25E144, U4 MAX3421E, U5 FE2.1-LQFP48, U6 ATtiny45-20PU, U7 DS1307Z+, U8 LM3940IS-3.3, U9 LD1117AS12TR, X1 27 MHz, X2 12 MHz, Y1 18.432 MHz, Y2 32768 Hz, Y3 4.433619 MHz

Commit message: update pcb rev.A
Parts:
- removed Q1: IRLML6402, Package_TO_SOT_SMD:SOT-23
- removed R7: 4.7k, Resistor_SMD:R_0603_1608Metric_Pad0.98x0.95mm_HandSolder
- added J18: ESP-01, Connector_PinSocket_2.54mm:PinSocket_2x04_P2.54mm_Vertical, F.Cu at (125.0, 134.3)
Connections:
- J1 pad 5: +5V_JOY -> (no net)
- J1 pad 7: Net-(J1-Pad7) -> +5V_JOY
- J3 pad 5: +5V_JOY -> (no net)
- J3 pad 7: Net-(J1-Pad7) -> +5V_JOY
- U5 pad 47: GND -> (no net)
Routing:
- net /RX_FPGA: track 63.1 -> 117.2 mm, vias 5 -> 7
- net /RST: track 174.4 -> 226.6 mm, vias 13 -> 15
- net Net-(J1-Pad7): track 19.4 -> 0.00 mm
- net /CONF_DCLK: track 101.8 -> 85.3 mm, vias 3 -> 2
- net +3V3: track 729.1 -> 736.2 mm
- net /TX_FPGA: track 153.3 -> 157.9 mm, vias 7 -> 6
- net +5V_JOY: track 22.2 -> 18.5 mm, vias 1 -> 0
- net /~LED_ARM: track 55.2 -> 53.0 mm
- net GND: track 537.6 -> 537.5 mm, vias 387 -> 386

Commit message: update pcb rev.A
Parts:
- R38: value x -> 0

Commit message: update pcb rev.A
Parts:
- H1, H2, H3, H4: footprint MountingHole:MountingHole_2.5mm -> MountingHole:MountingHole_2.7mm_M2.5_DIN965
- moved J18 0.20 mm to (125.2, 134.3)
- moved J4 0.10 mm to (127.5, 54.7)
Routing:
- net Net-(C11-Pad2): track 11.6 -> 12.3 mm
