File: pcb/rev.A/mist1010.kicad_pcb (KiCad board)
At the start: 2 copper layers, 100 x 100 mm, 241 parts, among them J1 Conn_02x05_Odd_Even, J10 TE 041021-4, J11 Conn_01x03, J12 Conn_01x04, J13 Conn_02x05_Odd_Even, J14 Conn_02x05_Odd_Even, J15 Conn_01x04, J16 MEM2055-00-190-01-A, J17 Conn_01x04, J18 ESP-01, J2 USB_B_Micro, J3 Conn_02x05_Odd_Even, J4 PJ-320, J5 USB_A, J6 USB_A, J7 USB_A, J8 USB_A, J9 DB15_Female_HighDensity_Mount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, Q2 IRLML6402, Q3 BC817, Q4 BC817, SW1 Jumper / Pin header 1x2 Pitch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, SW2 SW_DIP_x02, SW3 SW_Push, SW4 SW_Push, SW5 SW_Push, U1 MT48LC16M16A2, U10 LD1117AS25TR, U11 AD724, U2 AT91SAM7S256-AU, U3 EP3C25E144, U4 MAX3421E, U5 FE2.1-LQFP48, U6 ATtiny45-20PU, U7 DS1307Z+, U8 LM3940IS-3.3, U9 LD1117AS12TR, X1 27 MHz, X2 12 MHz, Y1 18.432 MHz, Y2 32768 Hz, Y3 4.433619 MHz

Commit message: update pcb rev.A
Parts:
- added LOGO1: graphic, my:black-mage-6.7x9.5, F.Cu at (158.7, 101.7)
- H1, H2, H3, H4: footprint MountingHole:MountingHole_2.7mm_M2.5_DIN965 -> MountingHole:MountingHole_3.2mm_M3_ISO14580
- moved J18 8.38 mm to (132.7, 130.8), turned to 0 degrees
- moved R45 5.50 mm to (129.5, 145.3)
- moved J4 0.20 mm to (127.7, 54.7)
- moved J7 0.10 mm to (184.0, 59.6)
- moved J8 0.10 mm to (193.8, 59.6)
Routing:
- net +3V3: track 736.3 -> 726.5 mm
- net /RX_FPGA: track 117.4 -> 125.9 mm, vias 7 -> 8
- net /~LED_ARM: track 53.0 -> 61.4 mm
- net Net-(C11-Pad2): track 12.3 -> 13.5 mm
- net /TX_FPGA: track 158.1 -> 158.6 mm
- net /RST: track 226.7 -> 226.3 mm, vias 15 -> 14
