File: pcb/rev.A/mist1010.kicad_sch (KiCad schematic)
At the start: 207 parts, among them J1 Conn_02x05_Odd_Even, J10 TE 041021-4, J11 Conn_01x03, J12 Conn_01x04, J13 Conn_02x05_Odd_Even, J14 Conn_02x05_Odd_Even, J15 Conn_01x04, J16 MEM2055-00-190-01-A, J17 Conn_01x04, J2 USB_B_Micro, J3 Conn_02x05_Odd_Even, J4 PJ-320D, J5 USB_A, J6 USB_A, J7 USB_A, J8 USB_A, J9 DB15_Female_HighDensity_Mount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, Q1 IRLML6402, Q2 IRLML6402, Q3 BC817, Q4 BC817, SW1 Jumper / Pin header 1x2 Pitch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, SW2 SW_DIP_x02, SW3 SW_Push, SW4 SW_Push, SW5 SW_Push, U1 MT48LC16M16A2, U10 LD1117AS25TR, U2 AT91SAM7S256-AU, U3 EP3C25E144, U4 MAX3421E, U5 FE2.1-LQFP48, U6 ATtiny45-20PU, U7 DS1307Z+, U8 LM3940IS-3.3, U9 LD1117AS12TR, X1 27 MHz, X2 12 MHz, Y1 18.432 MHz, Y2 32768 Hz

Commit message: update pcb rev.A
Parts:
- D1: value LED_RED -> LED_Red
- D2: value LED_YELLOW -> LED_Yellow
- D3: value LED_GREEN -> LED_Green
- J4: value PJ-320D -> PJ-320
- U7: ValueAlt (none) -> M41T56
Connections:
- net GND: now also J11.1 (Pin_1); no longer J11.3 (Pin_3)
- net TAPE_OUT: now also J11.3 (Pin_3); no longer J11.1 (Pin_1)
Changed lines of the file:
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@@
     (stroke (width 0.1524) (type solid) (color 0 0 0 0))
   )
-  (bus_entry (at 245.745 262.89) (size 2.54 2.54)
+  (bus_entry (at 245.745 265.43) (size 2.54 2.54)
     (stroke (width 0.1524) (type solid) (color 0 0 0 0))
   )
-  (bus_entry (at 245.745 265.43) (size 2.54 2.54)
+  (bus_entry (at 245.745 267.97) (size 2.54 2.54)
     (stroke (width 0.1524) (type solid) (color 0 0 0 0))
   )
@@
     (stroke (width 0) (type solid) (color 0 0 0 0))
   )
-  (wire (pts (xy 248.285 265.43) (xy 255.905 265.43))
+  (wire (pts (xy 248.285 267.97) (xy 255.905 267.97))
     (stroke (width 0) (type solid) (color 0 0 0 0))
   )
-  (wire (pts (xy 248.285 267.97) (xy 255.905 267.97))
+  (wire (pts (xy 248.285 270.51) (xy 255.905 270.51))
     (stroke (width 0) (type solid) (color 0 0 0 0))
   )
@@
     (effects (font (size 1 1)) (justify right bottom))
   )
-  (label "TAPE_OUT" (at 248.285 265.43 0)
+  (label "TAPE_IN" (at 248.285 267.97 0)
     (effects (font (size 1 1)) (justify left bottom))
   )
-  (label "TAPE_IN" (at 248.285 267.97 0)
+  (label "TAPE_OUT" (at 248.285 270.51 0)
     (effects (font (size 1 1)) (justify left bottom))
   )
@@
     (pin "1")
   )
-  (symbol (lib_id "power:GND") (at 255.905 270.51 270) (unit 1)
+  (symbol (lib_id "power:GND") (at 255.905 265.43 270) (unit 1)
     (in_bom yes) (on_board yes)
-    (property "Reference" "#PWR069" (id 0) (at 249.555 270.51 0)
+    (property "Reference" "#PWR069" (id 0) (at 249.555 265.43 0)
       (effects (font (size 1 1)) hide)
     )
-    (property "Value" "GND" (id 1) (at 250.3106 270.51 90)
+    (property "Value" "GND" (id 1) (at 250.3106 265.43 90)
       (effects (font (size 1 1)))
     )
-    (property "Footprint" "" (id 2) (at 255.905 270.51 0)
+    (property "Footprint" "" (id 2) (at 255.905 265.43 0)
       (effects (font (size 1.27 1.27)) hide)
     )
-    (property "Datasheet" "" (id 3) (at 255.905 270.51 0)
+    (property "Datasheet" "" (id 3) (at 255.905 265.43 0)
       (effects (font (size 1.27 1.27)) hide)
     )
@@
       (effects (font (size 1 1)))
     )
-    (property "Value" "LED_RED" (id 1) (at 489.585 264.16 90)
+    (property "Value" "LED_Red" (id 1) (at 492.76 264.16 90)
       (effects (font (size 1 1)))
     )
@@
       (effects (font (size 1 1)))
     )
-    (property "Value" "LED_YELLOW" (id 1) (at 500.38 264.16 90)
+    (property "Value" "LED_Yellow" (id 1) (at 501.65 264.16 90)
       (effects (font (size 1 1)))
     )
@@
       (effects (font (size 1 1)))
     )
-    (property "Value" "LED_GREEN" (id 1) (at 512.445 264.16 90)
+    (property "Value" "LED_Green" (id 1) (at 511.175 264.16 90)
       (effects (font (size 1 1)))
     )
@@
       (effects (font (size 1 1)) (justify right))
     )
-    (property "Value" "PJ-320D" (id 1) (at 494.157 93.1164 0)
+    (property "Value" "PJ-320" (id 1) (at 494.157 93.1164 0)
       (effects (font (size 1 1)) (justify right) hide)
     )
@@
       (effects (font (size 1 1)) (justify left))
     )
-    (property "Value" "DS1307Z+" (id 1) (at 377.825 285.7499 0)
+    (property "Value" "DS1307Z+" (id 1) (at 378.46 284.4799 0)
       (effects (font (size 1 1)) (justify left))
     )
@@
       (effects (font (size 1.27 1.27)) hide)
     )
+    (property "ValueAlt" "M41T56" (id 4) (at 381.635 285.75 0)
+      (effects (font (size 1 1)))
+    )
     (pin "1")
     (pin "2")
@@
     )
     (path "/7a2ff5d6-c068-4fe1-be7f-dcaf94f09902"
-      (reference "D1") (unit 1) (value "LED_RED") (footprint "LED_THT:LED_D3.0mm_Horizontal_O1.27mm_Z6.0mm")
+      (reference "D1") (unit 1) (value "LED_Red") (footprint "LED_THT:LED_D3.0mm_Horizontal_O1.27mm_Z6.0mm")
     )
     (path "/35b42faf-4604-4a4f-a642-c4bb2437cffa"
-      (reference "D2") (unit 1) (value "LED_YELLOW") (footprint "LED_THT:LED_D3.0mm_Horizontal_O1.27mm_Z6.0mm")
+      (reference "D2") (unit 1) (value "LED_Yellow") (footprint "LED_THT:LED_D3.0mm_Horizontal_O1.27mm_Z6.0mm")
     )
     (path "/a1d9b023-ff68-46c4-9dd0-0d3c73e90c6e"
-      (reference "D3") (unit 1) (value "LED_GREEN") (footprint "LED_THT:LED_D3.0mm_Horizontal_O1.27mm_Z6.0mm")
+      (reference "D3") (unit 1) (value "LED_Green") (footprint "LED_THT:LED_D3.0mm_Horizontal_O1.27mm_Z6.0mm")
     )
     (path "/a1f54365-abc1-43bd-90c1-dce8aa351571"
@@
     )
     (path "/7c2b712f-638f-4128-8ea8-d02c4be413f5"
-      (reference "J4") (unit 1) (value "PJ-320D") (footprint "my:PJ-320A_D")
+      (reference "J4") (unit 1) (value "PJ-320") (footprint "my:PJ-320A_D")
     )
     (path "/383290e8-a322-486f-9546-f4c35ea08e7e"

Commit message: update pcb rev.A
Parts:
- added C75, C76: 10u, Capacitor_SMD:C_0805_2012Metric_Pad1.18x1.45mm_HandSolder, symbol Device:C
- added C77, C78, C79: 100n, Capacitor_SMD:C_0603_1608Metric_Pad1.08x0.95mm_HandSolder, symbol Device:C
- added C80: 220u, Capacitor_Tantalum_SMD:CP_EIA-7343-31_Kemet-D, symbol Device:CP
- added C81: 10p, Capacitor_SMD:C_0603_1608Metric_Pad1.08x0.95mm_HandSolder, symbol Device:C
- added L4: 1u, Inductor_SMD:L_0805_2012Metric_Pad1.15x1.40mm_HandSolder, symbol Device:L
- added R101, R102, R103, R89: 75, Resistor_SMD:R_0603_1608Metric_Pad0.98x0.95mm_HandSolder, symbol Device:R
- added R76, R83, R91: 1k, Resistor_SMD:R_0603_1608Metric_Pad0.98x0.95mm_HandSolder, symbol Device:R
- added R77, R78, R84, R85, R92, R93: 1.1k, Resistor_SMD:R_0603_1608Metric_Pad0.98x0.95mm_HandSolder, symbol Device:R
- added R79, R86, R94: 2.2k, Resistor_SMD:R_0603_1608Metric_Pad0.98x0.95mm_HandSolder, symbol Device:R
- added R80, R87, R95: 4.3k, Resistor_SMD:R_0603_1608Metric_Pad0.98x0.95mm_HandSolder, symbol Device:R
- added R81, R88, R96: 9.1k, Resistor_SMD:R_0603_1608Metric_Pad0.98x0.95mm_HandSolder, symbol Device:R
- added R82, R90, R97: 18k, Resistor_SMD:R_0603_1608Metric_Pad0.98x0.95mm_HandSolder, symbol Device:R
- added R98: 4.7M, Resistor_SMD:R_0603_1608Metric_Pad0.98x0.95mm_HandSolder, symbol Device:R
- added U11: AD724, Package_SO:SOIC-16W_7.5x10.3mm_P1.27mm, symbol ad724:AD724
- added Y3: 4.433619 MHz, Crystal:Crystal_SMD_5032-2Pin_5.0x3.2mm, symbol Device:Crystal
- J4: Desc (none) -> RPi pinout
Connections:
- net +5V: now also L4.1
- net GND: now also C75.1, C76.1, C81.2, R101.2, R102.2, R103.2, R98.1, U11.1 (STDN), U11.12 (SELECT), U11.13 (DGND), U11.2 (AGND), Y3.2
- net VGA_B0: now also R91.1, R92.1
- net VGA_B1: now also R93.1
- net VGA_B2: now also R94.1
- net VGA_B3: now also R95.1
- net VGA_B4: now also R96.1
- net VGA_B5: now also R97.1
- net VGA_G0: now also R83.1, R84.1
- net VGA_G1: now also R85.1
- net VGA_G2: now also R86.1
- net VGA_G3: now also R87.1
- net VGA_G4: now also R88.1
- net VGA_G5: now also R90.1
- net VGA_HS: now also U11.16 (HSYNC)
- net VGA_R0: now also R76.1, R77.1
- net VGA_R1: now also R78.1
- net VGA_R2: now also R79.1
- net VGA_R3: now also R80.1
- net VGA_R4: now also R81.1
- net VGA_R5: now also R82.1
- net VGA_VS: now also U11.15 (VSYNC)
- net Composite: now reaches J4.S
- net Composite: now also R89.1
- new net: C77.2, R101.1, R76.2, R77.2, R78.2, R79.2, R80.2, R81.2, R82.2
- new net: C79.2, R103.1, R91.2, R92.2, R93.2, R94.2, R95.2, R96.2, R97.2
- new net: C77.1, U11.6 (RIN)
- new net: C78.1, U11.7 (GIN)
- new net: C78.2, R102.1, R83.2, R84.2, R85.2, R86.2, R87.2, R88.2, R90.2
- new net: C80.2, R89.2
- new net: C80.1, U11.10 (COMP)
- new net: C81.1, R98.2, U11.3 (FIN), Y3.1
- new net: C75.2, C76.2, L4.2, U11.14 (DVCC), U11.4 (AVCC), U11.5 (ENCD)
- new net: C79.1, U11.8 (BIN)
- no-connect marks 46 -> 47
Other:
- moved on the sheet: BT1, C11, C12, C13, C14, C17, C18, C19, C20, C21, C22, C23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

Commit message: update pcb rev.A
Parts:
- Y3: footprint Crystal:Crystal_SMD_5032-2Pin_5.0x3.2mm -> Crystal:Crystal_SMD_HC49-SD
Connections:
- net +5V_PAL: now reaches C75.2, C76.2, L4.2, U11.14 (DVCC), U11.4 (AVCC), U11.5 (ENCD)
Other:
- moved on the sheet: C30, C32, C33, C34, C35, C36, C37, C38, C75, C76, C77, C78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

Commit message: update pcb rev.A
Parts:
- removed Q1: IRLML6402, Package_TO_SOT_SMD:SOT-23, symbol Transistor_FET:IRLML6402
- removed R7: 4.7k, Resistor_SMD:R_0603_1608Metric_Pad0.98x0.95mm_HandSolder, symbol Device:R
- added J18: ESP-01, Connector_PinSocket_2.54mm:PinSocket_2x04_P2.54mm_Vertical, symbol Connector_Generic:Conn_02x04_Odd_Even
Connections:
- net +3V3: now also J18.4 (Pin_4), J18.8 (Pin_8)
- net +5V_JOY: now also J1.7 (Pin_7), J3.7 (Pin_7); no longer J1.5 (Pin_5), J3.5 (Pin_5)
- net GND: now also J18.1 (Pin_1); no longer U5.47 (LED6/NOP1)
- net RST: now also J18.6 (Pin_6)
- net RX_FPGA: now also J18.2 (Pin_2)
- net TX_FPGA: now also J18.7 (Pin_7)
- no-connect marks 47 -> 52
Other:
- note added: "AV out"
- note added: "Alternative microSD slot"
- note added: "Beeper"
- note added: "Buttons"
- note added: "Clock"
- note added: "Debug"
- note added: "FPGA"
- note added: "IO ARM controller"
- note added: "Joystick ports"
- note added: "LEDs"
- note added: "PAL encoder"
- note added: "Power"
- note added: "Power in / USB"
- note added: "RTC"
- note added: "SD card"
- note added: "SDRAM memory"
- note added: "Tape"
- note added: "USB controller and hub"
- note added: "USB host ports"
- note added: "VGA"
- note added: "WiFi"
- moved on the sheet: BT1, C1, C10, C11, C12, C13, C14, C15, C16, C17, C18, C19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

Commit message: update pcb rev.A
Parts:
- R38: value x -> 0
Other:
- moved on the sheet: C20, C21, J14, L3, R24, R69, R70, R71, R72

Commit message: update pcb rev.A
Parts:
- H1, H2, H3, H4: footprint MountingHole:MountingHole_2.5mm -> MountingHole:MountingHole_2.7mm_M2.5_DIN965
Changed lines of the file:
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@@
       (effects (font (size 1 1)) (justify left))
     )
-    (property "Footprint" "MountingHole:MountingHole_2.5mm" (id 2) (at 447.04 334.645 0)
+    (property "Footprint" "MountingHole:MountingHole_2.7mm_M2.5_DIN965" (id 2) (at 447.04 334.645 0)
       (effects (font (size 1.27 1.27)) hide)
     )
@@
       (effects (font (size 1 1)) (justify left))
     )
-    (property "Footprint" "MountingHole:MountingHole_2.5mm" (id 2) (at 447.04 340.36 0)
+    (property "Footprint" "MountingHole:MountingHole_2.7mm_M2.5_DIN965" (id 2) (at 447.04 340.36 0)
       (effects (font (size 1.27 1.27)) hide)
     )
@@
       (effects (font (size 1 1)) (justify left))
     )
-    (property "Footprint" "MountingHole:MountingHole_2.5mm" (id 2) (at 467.995 334.645 0)
+    (property "Footprint" "MountingHole:MountingHole_2.7mm_M2.5_DIN965" (id 2) (at 467.995 334.645 0)
       (effects (font (size 1.27 1.27)) hide)
     )
@@
       (effects (font (size 1 1)) (justify left))
     )
-    (property "Footprint" "MountingHole:MountingHole_2.5mm" (id 2) (at 467.995 340.36 0)
+    (property "Footprint" "MountingHole:MountingHole_2.7mm_M2.5_DIN965" (id 2) (at 467.995 340.36 0)
       (effects (font (size 1.27 1.27)) hide)
     )
@@
     )
     (path "/94f3dbfc-30e0-4568-a542-0adfd7440004"
-      (reference "H1") (unit 1) (value "MountingHole") (footprint "MountingHole:MountingHole_2.5mm")
+      (reference "H1") (unit 1) (value "MountingHole") (footprint "MountingHole:MountingHole_2.7mm_M2.5_DIN965")
     )
     (path "/2f8fe43d-0aef-44a9-b4e2-3b3365181bba"
-      (reference "H2") (unit 1) (value "MountingHole") (footprint "MountingHole:MountingHole_2.5mm")
+      (reference "H2") (unit 1) (value "MountingHole") (footprint "MountingHole:MountingHole_2.7mm_M2.5_DIN965")
     )
     (path "/387d9e43-d657-41ab-8d4a-96ecdbbfa1ca"
-      (reference "H3") (unit 1) (value "MountingHole") (footprint "MountingHole:MountingHole_2.5mm")
+      (reference "H3") (unit 1) (value "MountingHole") (footprint "MountingHole:MountingHole_2.7mm_M2.5_DIN965")
     )
     (path "/35d0454f-36ff-4f88-abfb-63c692ac59f4"
-      (reference "H4") (unit 1) (value "MountingHole") (footprint "MountingHole:MountingHole_2.5mm")
+      (reference "H4") (unit 1) (value "MountingHole") (footprint "MountingHole:MountingHole_2.7mm_M2.5_DIN965")
     )
     (path "/25e79a09-f4c4-4bda-a4ac-044ec6643c66"

Commit message: update pcb rev.A
Parts:
- added LOGO1: graphic, my:black-mage-6.7x9.5, symbol my:logo
- H1, H2, H3, H4: footprint MountingHole:MountingHole_2.7mm_M2.5_DIN965 -> MountingHole:MountingHole_3.2mm_M3_ISO14580
Changed lines of the file:
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@@
       (effects (font (size 1 1)) (justify left))
     )
-    (property "Footprint" "MountingHole:MountingHole_2.7mm_M2.5_DIN965" (id 2) (at 447.04 334.645 0)
+    (property "Footprint" "MountingHole:MountingHole_3.2mm_M3_ISO14580" (id 2) (at 447.04 334.645 0)
       (effects (font (size 1.27 1.27)) hide)
     )
@@
       (effects (font (size 1 1)) (justify left))
     )
-    (property "Footprint" "MountingHole:MountingHole_2.7mm_M2.5_DIN965" (id 2) (at 447.04 340.36 0)
+    (property "Footprint" "MountingHole:MountingHole_3.2mm_M3_ISO14580" (id 2) (at 447.04 340.36 0)
       (effects (font (size 1.27 1.27)) hide)
     )
@@
       (effects (font (size 1 1)) (justify left))
     )
-    (property "Footprint" "MountingHole:MountingHole_2.7mm_M2.5_DIN965" (id 2) (at 467.995 334.645 0)
+    (property "Footprint" "MountingHole:MountingHole_3.2mm_M3_ISO14580" (id 2) (at 467.995 334.645 0)
       (effects (font (size 1.27 1.27)) hide)
     )
@@
       (effects (font (size 1 1)) (justify left))
     )
-    (property "Footprint" "MountingHole:MountingHole_2.7mm_M2.5_DIN965" (id 2) (at 467.995 340.36 0)
+    (property "Footprint" "MountingHole:MountingHole_3.2mm_M3_ISO14580" (id 2) (at 467.995 340.36 0)
       (effects (font (size 1.27 1.27)) hide)
     )
@@
     (pin "2")
   )
+  (symbol (lib_id "my:logo") (at 431.8 337.185 0) (unit 1)
+    (in_bom yes) (on_board yes)
+    (property "Reference" "LOGO1" (id 0) (at 431.8 332.105 0)
+      (effects (font (size 1.27 1.27)) hide)
+    )
+    (property "Value" "graphic" (id 1) (at 431.8 343.535 0)
+      (effects (font (size 1.27 1.27)) hide)
+    )
+    (property "Footprint" "my:black-mage-6.7x9.5" (id 2) (at 431.8 342.265 0)
+      (effects (font (size 1.27 1.27)) hide)
+    )
+    (property "Datasheet" "~" (id 3) (at 432.562 342.265 0)
+      (effects (font (size 1.27 1.27)) hide)
+    )
+    (property "Desc" "Logo" (id 4) (at 431.8 339.09 0)
+      (effects (font (size 0.9906 0.9906)))
+    )
+  )
   (symbol (lib_id "Transistor_BJT:BC817") (at 154.94 256.54 0) (unit 1)
     (in_bom yes) (on_board yes)
@@
     )
     (path "/94f3dbfc-30e0-4568-a542-0adfd7440004"
-      (reference "H1") (unit 1) (value "MountingHole") (footprint "MountingHole:MountingHole_2.7mm_M2.5_DIN965")
+      (reference "H1") (unit 1) (value "MountingHole") (footprint "MountingHole:MountingHole_3.2mm_M3_ISO14580")
     )
     (path "/2f8fe43d-0aef-44a9-b4e2-3b3365181bba"
-      (reference "H2") (unit 1) (value "MountingHole") (footprint "MountingHole:MountingHole_2.7mm_M2.5_DIN965")
+      (reference "H2") (unit 1) (value "MountingHole") (footprint "MountingHole:MountingHole_3.2mm_M3_ISO14580")
     )
     (path "/387d9e43-d657-41ab-8d4a-96ecdbbfa1ca"
-      (reference "H3") (unit 1) (value "MountingHole") (footprint "MountingHole:MountingHole_2.7mm_M2.5_DIN965")
+      (reference "H3") (unit 1) (value "MountingHole") (footprint "MountingHole:MountingHole_3.2mm_M3_ISO14580")
     )
     (path "/35d0454f-36ff-4f88-abfb-63c692ac59f4"
-      (reference "H4") (unit 1) (value "MountingHole") (footprint "MountingHole:MountingHole_2.7mm_M2.5_DIN965")
+      (reference "H4") (unit 1) (value "MountingHole") (footprint "MountingHole:MountingHole_3.2mm_M3_ISO14580")
     )
     (path "/25e79a09-f4c4-4bda-a4ac-044ec6643c66"
@@
       (reference "L4") (unit 1) (value "1u") (footprint "Inductor_SMD:L_0805_2012Metric_Pad1.15x1.40mm_HandSolder")
     )
+    (path "/74bc78de-3bc3-4ca2-a941-3aa58a86950f"
+      (reference "LOGO1") (unit 1) (value "graphic") (footprint "my:black-mage-6.7x9.5")
+    )
     (path "/98f5b6b3-1608-46ad-a2ca-a387b7ba8f9e"

Commit message: update pcb rev.A
Parts:
- N1: value G738 -> G738 or G706
Changed lines of the file:
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@@
       (effects (font (size 1 1)) (justify left) hide)
     )
-    (property "Value" "G738" (id 1) (at 487.68 343.8524 0)
+    (property "Value" "G738 or G706" (id 1) (at 487.045 343.8524 0)
       (effects (font (size 1 1)) (justify left))
     )
@@
     )
     (path "/b487b0a1-b165-408b-b378-148f08d7f761"
-      (reference "N1") (unit 1) (value "G738") (footprint "")
+      (reference "N1") (unit 1) (value "G738 or G706") (footprint "")
     )
     (path "/ce695809-036d-4301-b0c8-a43459904e3a"
