File: pcb_covers/rev.A/mist1010_covers.kicad_pcb (KiCad board)
At the start: 2 copper layers, 133.5 x 61.5 mm, 16 parts, among them J10 TE 041021-4, J2 USB_B_Micro, J4 PJ-320D, J5 USB_A, J6 USB_A, J7 USB_A, J8 USB_A, J9 DB15_Female_HighDensity_Mount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, SW3 SW_Push, SW4 SW_Push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

Commit message: update pcb rev.A
Parts:
- removed D1: LED_RED, LED_THT:LED_D3.0mm_Horizontal_O1.27mm_Z6.0mm
- removed D2: LED_YELLOW, LED_THT:LED_D3.0mm_Horizontal_O1.27mm_Z6.0mm
- removed D3: LED_GREEN, LED_THT:LED_D3.0mm_Horizontal_O1.27mm_Z6.0mm
- removed J10 (x2): TE 041021-4, my:SD_TE_2041021-mod
- removed J2: USB_B_Micro, Connector_USB:USB_Micro-B_Molex-105017-0001
- removed J4: PJ-320D, my:PJ-320A_D
- removed J5, J6 (x2), J7, J8: USB_A, Connector_USB:USB_A_Wuerth_614004134726_Horizontal
- removed J9: DB15_Female_HighDensity_MountingHoles, Connector_Dsub:DSUB-15-HD_Female_Horizontal_P2.29x1.98mm_EdgePinOffset3.03mm_Housed_MountingHolesOffset4.94mm
- removed SW3, SW4, SW5: SW_Push, Button_Switch_THT:SW_Tactile_SPST_Angled_PTS645Vx58-2LFS
- added G***: LOGO, my:black-mage, B.Cu at (144.0, 102.5)
Routing:
- net COMMON: vias 0 -> 1
- net (no net): vias 1 -> 0
- added copper zone on B.Cu, net COMMON
- added copper zone on F.Cu, net COMMON
Other:
- outline, holes or cut-outs redrawn
- board text added: "JLCJLCJLCJLC"
- board text added: "MIST.1010 Back cover Rev.A"
- board text added: "MIST.1010 Front cover Rev.A"

Commit message: update pcb rev.A
Changed lines of the file:
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@@
     (style (thickness 0.15) (arrow_length 1.27) (text_position_mode 0) (extension_height 0.58642) (extension_offset 0.5) keep_text_aligned)
   )
-  (via (at 144.5 63) (size 0.8) (drill 0.4) (layers "F.Cu" "B.Cu") (free) (net 1))
+  (via (at 144.5 63) (size 1.2) (drill 0.8) (layers "F.Cu" "B.Cu") (free) (net 1))
   (zone (net 1) (net_name "COMMON") (layers F&B.Cu) (hatch edge 0.508)
     (connect_pads (clearance 0.508))

Commit message: update pcb rev.A
Other:
- outline, holes or cut-outs redrawn
Changed lines of the file:
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@@
   (gr_line (start 77.75 91) (end 77.75 61.5) (layer "Edge.Cuts") (width 0.1))
   (gr_line (start 77.75 123) (end 77.75 93.5) (layer "Edge.Cuts") (width 0.1))
-  (gr_line (start 129.5 91) (end 77.75 91) (layer "Edge.Cuts") (width 0.1))
+  (gr_line (start 135.5 91) (end 77.75 91) (layer "Edge.Cuts") (width 0.1))
   (gr_circle (center 122.7 72.1) (end 125.7 72.1) (layer "Edge.Cuts") (width 0.1) (fill none))
   (gr_circle (center 201.950784 88.732172) (end 200.550784 88.732172) (layer "Edge.Cuts") (width 0.1) (fill none))
@@
   (gr_circle (center 201.950784 63.732172) (end 200.550784 63.732172) (layer "Edge.Cuts") (width 0.1) (fill none))
   (gr_circle (center 87.049216 88.75) (end 88.449216 88.75) (layer "Edge.Cuts") (width 0.1) (fill none))
-  (gr_line (start 77.75 93.5) (end 129.5 93.5) (layer "Edge.Cuts") (width 0.1))
+  (gr_line (start 77.75 93.5) (end 135.5 93.5) (layer "Edge.Cuts") (width 0.1))
   (gr_arc (start 90.298331 83.982975) (end 90.049217 85.514344) (angle -100.8510762) (layer "Edge.Cuts") (width 0.1))
   (gr_arc (start 138.592462 81.759668) (end 138.035539 83.9) (angle 67.87145488) (layer "Edge.Cuts") (width 0.1))
@@
   (gr_rect (start 176.2 71.4) (end 182.2 85.4) (layer "Edge.Cuts") (width 0.1) (fill none))
   (gr_line (start 82.249216 69.085539) (end 82.249217 83.450003) (layer "Edge.Cuts") (width 0.1))
-  (gr_line (start 211.25 91) (end 159.5 91) (layer "Edge.Cuts") (width 0.1))
+  (gr_line (start 211.25 91) (end 153.5 91) (layer "Edge.Cuts") (width 0.1))
   (gr_circle (center 98.36 112.6) (end 99.91 112.6) (layer "Edge.Cuts") (width 0.1) (fill none))
   (gr_line (start 211.25 61.5) (end 211.25 91) (layer "Edge.Cuts") (width 0.1))
   (gr_rect (start 96.95 71.4) (end 102.95 85.4) (layer "Edge.Cuts") (width 0.1) (fill none))
-  (gr_line (start 159.5 93.5) (end 211.25 93.5) (layer "Edge.Cuts") (width 0.1))
+  (gr_line (start 153.5 93.5) (end 211.25 93.5) (layer "Edge.Cuts") (width 0.1))
   (gr_line (start 211.25 123) (end 77.75 123) (layer "Edge.Cuts") (width 0.1))
   (gr_line (start 138.035539 83.9) (end 152.400003 83.899999) (layer "Edge.Cuts") (width 0.1))
@@
   (gr_arc (start 90.298491 68.481185) (end 91.849216 68.525) (angle -100.8649601) (layer "Edge.Cuts") (width 0.1))
   (gr_circle (center 111.6 112.6) (end 113.15 112.6) (layer "Edge.Cuts") (width 0.1) (fill none))
-  (gr_line (start 159.5 93.5) (end 159.5 91) (layer "Edge.Cuts") (width 0.1))
+  (gr_line (start 153.5 93.5) (end 153.5 91) (layer "Edge.Cuts") (width 0.1))
   (gr_circle (center 165.175 113.3) (end 168.325 113.3) (layer "Edge.Cuts") (width 0.1) (fill none))
-  (gr_line (start 129.5 91) (end 129.5 93.5) (layer "Edge.Cuts") (width 0.1))
+  (gr_line (start 135.5 91) (end 135.5 93.5) (layer "Edge.Cuts") (width 0.1))
   (gr_rect (start 129.7 117.4) (end 159.1 114.3) (layer "Edge.Cuts") (width 0.1) (fill none))
   (gr_line (start 91.849216 68.525) (end 91.849216 83.939344) (layer "Edge.Cuts") (width 0.1))
@@
     (style (thickness 0.15) (arrow_length 1.27) (text_position_mode 0) (extension_height 0.58642) (extension_offset 0.5) keep_text_aligned)
   )
-  (via (at 144.5 63) (size 1.2) (drill 0.8) (layers "F.Cu" "B.Cu") (free) (net 1))
+  (via (at 144.5 92.3) (size 1.2) (drill 0.8) (layers "F.Cu" "B.Cu") (free) (net 1))
   (zone (net 1) (net_name "COMMON") (layers F&B.Cu) (hatch edge 0.508)
     (connect_pads (clearance 0.508))

Commit message: update pcb rev.A
Other:
- board size 133.5 x 61.5 mm -> 133.5 x 62 mm

Commit message: update pcb rev.A
Other:
- board size 133.5 x 62 mm -> 134.4 x 62 mm

Commit message: update pcb rev.A
Other:
- outline, holes or cut-outs redrawn
Changed lines of the file:
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@@
   )
   (gr_arc (start 157.01 78.65) (end 157.01 81.65) (angle -180) (layer "B.SilkS") (width 0.4))
-  (gr_circle (center 168.2 72.3) (end 173.3 72.3) (layer "B.SilkS") (width 0.4) (fill none))
+  (gr_circle (center 168.2 72.3) (end 171.95 72.3) (layer "B.SilkS") (width 0.4) (fill none))
   (gr_arc (start 198.700885 68.266794) (end 198.949999 66.735425) (angle -100.8510762) (layer "B.SilkS") (width 0.4))
   (gr_line (start 205.7 84.46423) (end 198.949999 85.29977) (layer "B.SilkS") (width 0.4))
@@
   (gr_circle (center 201.95 88.5) (end 203.35 88.5) (layer "Edge.Cuts") (width 0.1) (fill none))
   (gr_line (start 77.3 61) (end 211.7 61) (layer "Edge.Cuts") (width 0.1))
-  (gr_circle (center 168.2 72.3) (end 173.3 72.3) (layer "Edge.Cuts") (width 0.1) (fill none))
+  (gr_circle (center 168.2 72.3) (end 171.95 72.3) (layer "Edge.Cuts") (width 0.1) (fill none))
   (gr_circle (center 178.675 112.9) (end 181.825 112.9) (layer "Edge.Cuts") (width 0.1) (fill none))
   (gr_line (start 83.299216 84.500231) (end 90.049217 85.264575) (layer "Edge.Cuts") (width 0.1))
@@
     (effects (font (size 1.1 0.8) (thickness 0.14)) (justify mirror))
   )
-  (gr_text "Power" (at 168.2 65.1) (layer "B.SilkS")
+  (gr_text "Power" (at 168.2 66.6) (layer "B.SilkS")
     (effects (font (size 2 1.2) (thickness 0.2)) (justify mirror))
   )
